File: IRF2104_MOSFET_Driver-master/IRF2104_MOSFET_Driver-master/IRF2104 Driver.kicad_pcb (KiCad board)
At the start: 2 copper layers, 66 x 64.8 mm, 26 parts, among them J1 Screw_Terminal_01x02, J2 Conn_01x03_Female, J3 Conn_01x03_Male, J4 Screw_Terminal_01x03, Q1 IRF3205, Q2 IRF3205, Q3 IRF3205, Q4 IRF3205, U1 IR2104, U2 IR2104

Commit message: Resistor issue fixed
Parts:
- moved R12 8.35 mm to (120.0, 100.3), turned to 270 degrees
- moved R13 8.28 mm to (111.1, 125.1), turned to 270 degrees
Routing:
- net Net-(J2-Pad3): track 15.1 -> 4.67 mm
- net Net-(J2-Pad2): track 24.6 -> 16.6 mm
- net Net-(D4-Pad1): track 14.8 -> 22.5 mm
- net Net-(D5-Pad1): track 16.6 -> 22.3 mm
Changed lines of the file:
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@@
     (thickness 1.6)
     (drawings 8)
-    (tracks 135)
+    (tracks 130)
     (zones 0)
     (modules 26)
@@
   )
   (setup
-    (last_trace_width 1)
+    (last_trace_width 0.5)
     (user_trace_width 0.5)
     (user_trace_width 1)
@@
   )
   (module Resistor_THT:R_Axial_DIN0207_L6.3mm_D2.5mm_P7.62mm_Horizontal (layer F.Cu)
-    (at 128.27 101.6 180)
+    (at 120.015 100.33 270)
     (descr "Resistor, Axial_DIN0207 series, Axial, Horizontal, pin pitch=7.62mm, 0.25W = 1/4W, length*diameter=6.3*2.5mm^2, http://cdn-reichelt.de/documents/datenblatt/B400/1_4W%23YAG.pdf")
     (tags "Resistor Axial_DIN0207 series Axial Horizontal pin pitch 7.62mm 0.25W = 1/4W length 6.3mm diameter 2.5mm")
-    (fp_text reference R12 (at 3.81 -2.37 180) (layer F.SilkS)
-      (effects (font (size 1 1) (thickness 0.15)))
-    )
-    (fp_text value 1k (at 3.81 2.37 180) (layer F.Fab)
+    (fp_text reference R12 (at 3.81 -2.37 270) (layer F.SilkS)
+      (effects (font (size 1 1) (thickness 0.15)))
+    )
+    (fp_text value 1k (at 3.81 2.37 270) (layer F.Fab)
       (effects (font (size 1 1) (thickness 0.15)))
     )
@@
     (fp_line (start 8.67 1.5) (end 8.67 -1.5) (layer F.CrtYd) (width 0.05))
     (fp_line (start 8.67 -1.5) (end -1.05 -1.5) (layer F.CrtYd) (width 0.05))
-    (fp_text user %R (at 3.81 0 180) (layer F.Fab)
-      (effects (font (size 1 1) (thickness 0.15)))
-    )
-    (pad 1 thru_hole circle (at 0 0 180) (size 1.6 1.6) (drill 0.8) (layers *.Cu *.Mask)
+    (fp_text user %R (at 3.81 0 270) (layer F.Fab)
+      (effects (font (size 1 1) (thickness 0.15)))
+    )
+    (pad 1 thru_hole circle (at 0 0 270) (size 1.6 1.6) (drill 0.8) (layers *.Cu *.Mask)
       (net 9 "Net-(D5-Pad1)"))
-    (pad 2 thru_hole oval (at 7.62 0 180) (size 1.6 1.6) (drill 0.8) (layers *.Cu *.Mask)
+    (pad 2 thru_hole oval (at 7.62 0 270) (size 1.6 1.6) (drill 0.8) (layers *.Cu *.Mask)
       (net 11 "Net-(J2-Pad3)"))
     (model ${KISYS3DMOD}/Resistor_THT.3dshapes/R_Axial_DIN0207_L6.3mm_D2.5mm_P7.62mm_Horizontal.wrl
@@
   )
   (module Resistor_THT:R_Axial_DIN0207_L6.3mm_D2.5mm_P7.62mm_Horizontal (layer F.Cu)
-    (at 111.76 133.35)
+    (at 111.125 125.095 270)
     (descr "Resistor, Axial_DIN0207 series, Axial, Horizontal, pin pitch=7.62mm, 0.25W = 1/4W, length*diameter=6.3*2.5mm^2, http://cdn-reichelt.de/documents/datenblatt/B400/1_4W%23YAG.pdf")
     (tags "Resistor Axial_DIN0207 series Axial Horizontal pin pitch 7.62mm 0.25W = 1/4W length 6.3mm diameter 2.5mm")
-    (fp_text reference R13 (at 3.81 -2.37) (layer F.SilkS)
-      (effects (font (size 1 1) (thickness 0.15)))
-    )
-    (fp_text value 1k (at 3.81 2.37) (layer F.Fab)
+    (fp_text reference R13 (at 3.81 -2.37 90) (layer F.SilkS)
+      (effects (font (size 1 1) (thickness 0.15)))
+    )
+    (fp_text value 1k (at 3.81 2.37 90) (layer F.Fab)
       (effects (font (size 1 1) (thickness 0.15)))
     )
@@
     (fp_line (start 8.67 1.5) (end 8.67 -1.5) (layer F.CrtYd) (width 0.05))
     (fp_line (start 8.67 -1.5) (end -1.05 -1.5) (layer F.CrtYd) (width 0.05))
-    (fp_text user %R (at 3.81 0) (layer F.Fab)
-      (effects (font (size 1 1) (thickness 0.15)))
-    )
-    (pad 1 thru_hole circle (at 0 0) (size 1.6 1.6) (drill 0.8) (layers *.Cu *.Mask)
+    (fp_text user %R (at 3.81 0 90) (layer F.Fab)
+      (effects (font (size 1 1) (thickness 0.15)))
+    )
+    (pad 1 thru_hole circle (at 0 0 270) (size 1.6 1.6) (drill 0.8) (layers *.Cu *.Mask)
       (net 10 "Net-(J2-Pad2)"))
-    (pad 2 thru_hole oval (at 7.62 0) (size 1.6 1.6) (drill 0.8) (layers *.Cu *.Mask)
+    (pad 2 thru_hole oval (at 7.62 0 270) (size 1.6 1.6) (drill 0.8) (layers *.Cu *.Mask)
       (net 8 "Net-(D4-Pad1)"))
     (model ${KISYS3DMOD}/Resistor_THT.3dshapes/R_Axial_DIN0207_L6.3mm_D2.5mm_P7.62mm_Horizontal.wrl
@@
   (segment (start 132.05 98.02) (end 134.35 98.02) (width 1.5) (layer B.Cu) (net 7))
   (segment (start 134.35 98.02) (end 134.62 98.29) (width 1.5) (layer B.Cu) (net 7))
-  (segment (start 121.53 133.35) (end 121.85 133.03) (width 1) (layer B.Cu) (net 8))
-  (segment (start 119.38 133.35) (end 121.53 133.35) (width 1) (layer B.Cu) (net 8))
   (segment (start 134.62 110.49) (end 147.32 123.19) (width 1.5) (layer B.Cu) (net 7))
   (segment (start 134.62 110.49) (end 121.88 123.23) (width 1.5) (layer B.Cu) (net 7))
@@
   (segment (start 120.9 129.54) (end 121.85 130.49) (width 1) (layer B.Cu) (net 7))
   (segment (start 116.84 129.54) (end 120.9 129.54) (width 1) (layer B.Cu) (net 7))
-  (segment (start 114.3 140.44) (end 114.3 142.24) (width 1) (layer B.Cu) (net 8))
-  (segment (start 114.3 136.295998) (end 114.3 140.44) (width 1) (layer B.Cu) (net 8))
-  (segment (start 119.38 133.35) (end 117.245998 133.35) (width 1) (layer B.Cu) (net 8))
-  (segment (start 117.245998 133.35) (end 114.3 136.295998) (width 1) (layer B.Cu) (net 8))
-  (segment (start 131.82 100.33) (end 132.05 100.56) (width 1) (layer B.Cu) (net 9))
-  (segment (start 123.19 109.22) (end 123.429999 108.980001) (width 1) (layer B.Cu) (net 9))
-  (segment (start 127.13863 101.6) (end 128.27 101.6) (width 1) (layer B.Cu) (net 9))
-  (segment (start 124.865998 101.6) (end 127.13863 101.6) (width 1) (layer B.Cu) (net 9))
-  (segment (start 123.19 103.275998) (end 124.865998 101.6) (width 1) (layer B.Cu) (net 9))
-  (segment (start 123.19 109.22) (end 123.19 103.275998) (width 1) (layer B.Cu) (net 9))
-  (segment (start 129.31 100.56) (end 128.27 101.6) (width 1) (layer B.Cu) (net 9))
-  (segment (start 132.05 100.56) (end 129.31 100.56) (width 1) (layer B.Cu) (net 9))
+  (segment (start 111.44 133.03) (end 111.125 132.715) (width 1) (layer B.Cu) (net 8))
+  (segment (start 121.85 133.03) (end 111.44 133.03) (width 1) (layer B.Cu) (net 8))
+  (segment (start 113 142.24) (end 114.3 142.24) (width 1) (layer B.Cu) (net 8))
+  (segment (start 111.125 140.365) (end 113 142.24) (width 1) (layer B.Cu) (net 8))
+  (segment (start 111.125 132.715) (end 111.125 140.365) (width 1) (layer B.Cu) (net 8))
+  (segment (start 120.245 100.56) (end 120.015 100.33) (width 1) (layer B.Cu) (net 9))
+  (segment (start 132.05 100.56) (end 120.245 100.56) (width 1) (layer B.Cu) (net 9))
+  (segment (start 123.19 107.92) (end 123.19 109.22) (width 1) (layer B.Cu) (net 9))
+  (segment (start 123.19 104.63637) (end 123.19 107.92) (width 1) (layer B.Cu) (net 9))
+  (segment (start 120.015 101.46137) (end 123.19 104.63637) (width 1) (layer B.Cu) (net 9))
+  (segment (start 120.015 100.33) (end 120.015 101.46137) (width 1) (layer B.Cu) (net 9))
+  (segment (start 113.567919 114.53) (end 114.77 114.53) (width 1) (layer B.Cu) (net 10))
+  (segment (start 111.125 116.972919) (end 113.567919 114.53) (width 1) (layer B.Cu) (net 10))
+  (segment (start 111.125 125.095) (end 111.125 116.972919) (width 1) (layer B.Cu) (net 10))
   (segment (start 118.54 114.53) (end 118.58 114.57) (width 1) (layer B.Cu) (net 10))
   (segment (start 114.77 114.53) (end 118.54 114.53) (width 1) (layer B.Cu) (net 10))
-  (segment (start 113.567919 114.53) (end 114.77 114.53) (width 1) (layer B.Cu) (net 10))
-  (segment (start 111.76 116.337919) (end 113.567919 114.53) (width 1) (layer B.Cu) (net 10))
-  (segment (start 111.76 133.35) (end 111.76 116.337919) (width 1) (layer B.Cu) (net 10))
-  (segment (start 118.54 111.99) (end 118.58 112.03) (width 1) (layer B.Cu) (net 11))
-  (segment (start 114.77 111.99) (end 118.54 111.99) (width 1) (layer B.Cu) (net 11))
-  (segment (start 120.65 109.96) (end 120.65 101.6) (width 1) (layer B.Cu) (net 11))
-  (segment (start 118.58 112.03) (end 120.65 109.96) (width 1) (layer B.Cu) (net 11))
+  (segment (start 120.015 110.595) (end 118.58 112.03) (width 1) (layer B.Cu) (net 11))
+  (segment (start 120.015 107.95) (end 120.015 110.595) (width 1) (layer B.Cu) (net 11))
   (segment (start 152.15 87.63) (end 153.87 89.35) (width 1) (layer B.Cu) (net 12))
   (segment (start 149.86 87.63) (end 152.15 87.63) (width 1) (layer B.Cu) (net 12))
