File: mosfet driver.sch (KiCad schematic (older format))
At the start: 23 parts, among them J1 Screw_Terminal_01x03, J2 Screw_Terminal_01x02, J3 Conn_01x03_Male, Q1 IRF3205, Q2 IRF3205, Q3 IRF3205, Q4 IRF3205, U1 IR2104, U2 IR2104

Commit message: Input and output filters added
Changes suggested by Malhar implemented. Input and output filters added. Output for current sensor added. MOLEX connector outputs added. LED added. Switches added.
Parts:
- removed J1: Screw_Terminal_01x03, TerminalBlock_Phoenix:TerminalBlock_Phoenix_MKDS-3-3-5.08_1x03_P5.08mm_Horizontal, symbol Connector:Screw_Terminal_01x03
- removed R10, R3, R4, R9: 1K, Resistor_SMD:R_0805_2012Metric_Pad1.15x1.40mm_HandSolder, symbol Device:R
- added C10, C7, C8, C9: 1uF, Capacitor_THT:C_Disc_D3.4mm_W2.1mm_P2.50mm, symbol Device:C_Small
- added C11, C14, C15: 270uF/35V, Capacitor_THT:CP_Radial_D10.0mm_P2.50mm_P5.00mm, symbol Device:CP_Small
- added C12, C13, C3, C4, C5, C6: 0.1uF, Capacitor_THT:C_Disc_D3.4mm_W2.1mm_P2.50mm, symbol Device:C_Small
- added D4, D6: LED, LED_THT:LED_D3.0mm, symbol Device:LED
- added H1, H2, H3, H4: MountingHole, MountingHole:MountingHole_3.2mm_M3_Pad_Via, symbol Mechanical:MountingHole
- added J1, J4: PWR_IN, TerminalBlock_Phoenix:TerminalBlock_Phoenix_MKDS-1,5-2-5.08_1x02_P5.08mm_Horizontal, symbol Connector:Screw_Terminal_01x02
- added J5: Screw_Terminal_01x02, Connector_Molex:Molex_KK-396_A-41791-0002_1x02_P3.96mm_Vertical, symbol Connector:Screw_Terminal_01x02
- added R10, R3, R4, R6, R8, R9: 10, Resistor_THT:R_Axial_DIN0204_L3.6mm_D1.6mm_P5.08mm_Horizontal, symbol Device:R_Small
- added R11, R12: 1k, Resistor_THT:R_Axial_DIN0204_L3.6mm_D1.6mm_P5.08mm_Horizontal, symbol Device:R
- added SW1: SW_DIP_x01, Button_Switch_THT:SW_DIP_SPSTx01_Slide_6.7x4.1mm_W7.62mm_P2.54mm_LowProfile, symbol Switch:SW_DIP_x01
- D1, D3: footprint Diode_SMD:D_0603_1608Metric_Pad1.05x0.95mm_HandSolder -> Diode_THT:D_DO-35_SOD27_P7.62mm_Horizontal
- D2, D5: footprint Diode_SMD:D_SOD-323_HandSoldering -> Diode_THT:D_DO-35_SOD27_P7.62mm_Horizontal
- Q1, Q2, Q3, Q4: footprint mosfet_with_hest_sink:heatsink2 -> Heatsink:heatsinknew
- R1, R2, R5, R7: footprint Resistor_SMD:R_0805_2012Metric_Pad1.15x1.40mm_HandSolder -> Resistor_THT:R_Axial_DIN0204_L3.6mm_D1.6mm_P5.08mm_Horizontal
Connections:
- net labels removed: Power2
- wire segments 84 -> 120
Other:
- note added: "1n5822\n1n5819\n"
- note added: "22K\n"
- moved on the sheet: C1, C2

Commit message: Current Sensor placement solved
Switch for current sensor added for bypassing it whenever unnecessary. This board is also tailored for manufacturing in-house.
Parts:
- added SW2: SW_DIP_x01, Button_Switch_THT:SW_DIP_SPSTx01_Slide_6.7x4.1mm_W7.62mm_P2.54mm_LowProfile, symbol Switch:SW_DIP_x01
- H1, H2, H3, H4: symbol Mechanical:MountingHole -> mosfet-driver-rescue:MountingHole-Mechanical
- renumbered J5 to CS1
Connections:
- wire segments 120 -> 122
Other:
- moved on the sheet: CS1, D4, D6, J1, J4, R11, R12, SW1
